Commit message: added inertia to URDF (still needs work) and added gazebo and transmission xacros

File: motoman_mh5_support/urdf/mh5_macro.xacro (robot description, xacro)
@@ -1,5 +1,25 @@
 <?xml version="1.0" ?>
 <robot xmlns:xacro="http://ros.org/wiki/xacro">
+  <xacro:include filename="$(find motoman_mh5_support)/urdf/mh5.transmission.xacro" />
+  <xacro:include filename="$(find motoman_mh5_support)/urdf/mh5.gazebo.xacro" />
+  <xacro:macro name="cylinder_inertial" params="radius length mass *origin">
+    <inertial>
+      <mass value="${mass}" />
+      <xacro:insert_block name="origin" />
+      <inertia ixx="${0.0833333 * mass * (3 * radius * radius + length * length)}" ixy="0.0" ixz="0.0"
+        iyy="${0.0833333 * mass * (3 * radius * radius + length * length)}" iyz="0.0"
+        izz="${0.5 * mass * radius * radius}" />
+    </inertial>
+  </xacro:macro>
 	<xacro:macro name="motoman_mh5" params="prefix">
+    <!-- Inertia parameters -->
+    <!--TODO update all Mass parameters for the mh5 arm, these are all incorrect!!-->
+    <xacro:property name="base_mass" value="4.0" />
+    <xacro:property name="shoulder_mass" value="3.7000" />
+    <xacro:property name="upper_arm_mass" value="8.3930" />
+    <xacro:property name="forearm_mass" value="2.2750" />
+    <xacro:property name="wrist_1_mass" value="1.2190" />
+    <xacro:property name="wrist_2_mass" value="1.2190" />
+    <xacro:property name="wrist_3_mass" value="0.1879" />
 		<!-- link list -->
 		<link name="${prefix}base_link">
@@ -22,4 +42,7 @@
 				</material>
 			</collision>
+      <xacro:cylinder_inertial radius="0.06" length="0.05" mass="${base_mass}">
+        <origin xyz="0.0 0.0 0.0" rpy="0 0 0" />
+      </xacro:cylinder_inertial>
 		</link>
 		<link name="${prefix}link_s">
@@ -38,4 +61,7 @@
 				<material name="yellow"/>
 			</collision>
+      <xacro:cylinder_inertial radius="0.06" length="0.15" mass="${shoulder_mass}">
+        <origin xyz="0.0 0.0 0.0" rpy="0 0 0" />
+      </xacro:cylinder_inertial>
 		</link>
 		<link name="${prefix}link_l">
@@ -54,4 +80,7 @@
 				<material name="yellow"/>
 			</collision>
+      <xacro:cylinder_inertial radius="0.06" length="0.56" mass="${upper_arm_mass}">
+        <origin xyz="0.0 0.0 0.28" rpy="0 0 0" />
+      </xacro:cylinder_inertial>
 		</link>
 		<link name="${prefix}link_u">
@@ -70,4 +99,7 @@
 				<material name="yellow"/>
 			</collision>
+      <xacro:cylinder_inertial radius="0.06" length="0.5" mass="${forearm_mass}">
+        <origin xyz="0.0 0.0 0.25" rpy="0 0 0" />
+      </xacro:cylinder_inertial>
 		</link>
 		<link name="${prefix}link_r">
@@ -86,4 +118,7 @@
 				<material name="yellow"/>
 			</collision>
+      <xacro:cylinder_inertial radius="0.6" length="0.12" mass="${wrist_1_mass}">
+        <origin xyz="0.0 0.0 0.0" rpy="0 0 0" />
+      </xacro:cylinder_inertial>
 		</link>
 		<link name="${prefix}link_b">
@@ -102,4 +137,7 @@
 				<material name="yellow"/>
 			</collision>
+      <xacro:cylinder_inertial radius="0.6" length="0.12" mass="${wrist_2_mass}">
+        <origin xyz="0.0 0.0 0.0" rpy="0 0 0" />
+      </xacro:cylinder_inertial>
 		</link>
 		<link name="${prefix}link_t">
@@ -116,4 +154,7 @@
 				<material name="yellow"/>
 			</collision>
+      <xacro:cylinder_inertial radius="0.6" length="0.12" mass="${wrist_3_mass}">
+        <origin xyz="0.0 0.0 0.0" rpy="0 0 0" />
+      </xacro:cylinder_inertial>
 		</link>
 		<!-- end of link list -->
@@ -167,4 +208,6 @@
 		</joint>
 		<!-- end of joint list -->
+    <xacro:motoman_mh5_transmission prefix="${prefix}" />
+    <xacro:motoman_mh5_gazebo prefix="${prefix}" />
 	</xacro:macro>
 </robot>
