Commit message: added mh5l robot arm

File: motoman_mh5_support/urdf/mh5l_macro.xacro (robot description, xacro)
@@ -12,7 +12,7 @@
         </inertial>
     </xacro:macro>
-    <xacro:macro name="motoman_mh5" params="prefix">
+    <xacro:macro name="motoman_mh5l" params="prefix">
         <!-- Inertia parameters -->
-        <!--TODO update all Mass parameters for the mh5 arm, these are all incorrect!!-->
+        <!--TODO update all Mass parameters for the mh5l arm, these are all incorrect!!-->
         <xacro:property name="base_mass" value="4.0" />
         <xacro:property name="shoulder_mass" value="3.7000" />
@@ -25,20 +25,12 @@
         <link name="${prefix}base_link">
             <visual>
-                <origin rpy="0 0 3.14159"/>
                 <geometry>
-                    <mesh filename="package://motoman_mh5_support/meshes/mh5/visual/MH5_BASE_AXIS.stl" />
+                    <mesh filename="package://motoman_mh5_support/meshes/mh5l/visual/MH5L_BASE_AXIS.dae" />
                 </geometry>
-                <material name="blue">
-                    <color rgba="0 0 1 1"/>
-                </material>
             </visual>
             <collision>
-                <origin rpy="0 0 3.14159"/>
                 <geometry>
-                    <mesh filename="package://motoman_mh5_support/meshes/mh5/collision/MH5_BASE_AXIS.stl" />
+                    <mesh filename="package://motoman_mh5_support/meshes/mh5l/collision/MH5L_BASE_AXIS.stl" />
                 </geometry>
-                <material name="yellow">
-                    <color rgba="0 1 1 1"/>
-                </material>
             </collision>
             <xacro:cylinder_inertial radius="0.06" length="0.05" mass="${base_mass}">
@@ -49,15 +41,11 @@
             <visual>
                 <geometry>
-                    <mesh filename="package://motoman_mh5_support/meshes/mh5/visual/MH5_S_AXIS.stl"/>
+                    <mesh filename="package://motoman_mh5_support/meshes/mh5l/visual/MH5L_S_AXIS.dae"/>
                 </geometry>
-                <material name="silver">
-                    <color rgba="0.8 0.8 0.8 1"/>
-                </material>
             </visual>
             <collision>
                 <geometry>
-                    <mesh filename="package://motoman_mh5_support/meshes/mh5/collision/MH5_S_AXIS.stl" />
+                    <mesh filename="package://motoman_mh5_support/meshes/mh5l/collision/MH5L_S_AXIS.stl" />
                 </geometry>
-                <material name="yellow"/>
             </collision>
             <xacro:cylinder_inertial radius="0.06" length="0.15" mass="${shoulder_mass}">
@@ -67,16 +55,12 @@
         <link name="${prefix}link_l">
             <visual>
-                <!-- <origin rpy="1.57 3.1416 0" xyz="0 0 0"/> -->
                 <geometry>
-                    <mesh filename="package://motoman_mh5_support/meshes/mh5/visual/MH5_L_AXIS.stl"/>
+                    <mesh filename="package://motoman_mh5_support/meshes/mh5l/visual/MH5L_L_AXIS.dae"/>
                 </geometry>
-                <material name="blue"/>
             </visual>
             <collision>
-                <!-- <origin rpy="1.57 3.1416 0" xyz="0 0 0"/> -->
                 <geometry>
-                    <mesh filename="package://motoman_mh5_support/meshes/mh5/collision/MH5_L_AXIS.stl" />
+                    <mesh filename="package://motoman_mh5_support/meshes/mh5l/collision/MH5L_L_AXIS.stl" />
                 </geometry>
-                <material name="yellow"/>
             </collision>
             <xacro:cylinder_inertial radius="0.06" length="0.56" mass="${upper_arm_mass}">
@@ -86,16 +70,12 @@
         <link name="${prefix}link_u">
             <visual>
-                <!-- <origin rpy="1.57 -3.1415 0" xyz="0 0 0"/> -->
                 <geometry>
-                    <mesh filename="package://motoman_mh5_support/meshes/mh5/visual/MH5_U_AXIS.stl"/>
+                    <mesh filename="package://motoman_mh5_support/meshes/mh5l/visual/MH5L_U_AXIS.dae"/>
                 </geometry>
-                <material name="blue"/>
             </visual>
             <collision>
-                <!-- <origin rpy="1.57 -3.1415 0" xyz="0 0 0"/> -->
                 <geometry>
-                    <mesh filename="package://motoman_mh5_support/meshes/mh5/collision/MH5_U_AXIS.stl" />
+                    <mesh filename="package://motoman_mh5_support/meshes/mh5l/collision/MH5L_U_AXIS.stl" />
                 </geometry>
-                <material name="yellow"/>
             </collision>
             <xacro:cylinder_inertial radius="0.06" length="0.5" mass="${forearm_mass}">
@@ -105,16 +85,12 @@
         <link name="${prefix}link_r">
             <visual>
-                <!-- <origin rpy="0 0 3.1416" xyz="0 0 0"/> -->
                 <geometry>
-                    <mesh filename="package://motoman_mh5_support/meshes/mh5/visual/MH5_R_AXIS.stl"/>
+                    <mesh filename="package://motoman_mh5_support/meshes/mh5l/visual/MH5L_R_AXIS.dae"/>
                 </geometry>
-                <material name="silver"/>
             </visual>
             <collision>
-                <!-- <origin rpy="0 0 3.1416" xyz="0 0 0"/> -->
                 <geometry>
-                    <mesh filename="package://motoman_mh5_support/meshes/mh5/collision/MH5_R_AXIS.stl" />
+                    <mesh filename="package://motoman_mh5_support/meshes/mh5l/collision/MH5L_R_AXIS.stl" />
                 </geometry>
-                <material name="yellow"/>
             </collision>
             <xacro:cylinder_inertial radius="0.6" length="0.12" mass="${wrist_1_mass}">
@@ -124,16 +100,12 @@
 		<link name="${prefix}link_b">
 			<visual>
-				<!-- <origin rpy="-1.57 0 3.1416" xyz="0 0 0"/> -->
 				<geometry>
-					<mesh filename="package://motoman_mh5_support/meshes/mh5/visual/MH5_B_AXIS.stl"/>
+                    <mesh filename="package://motoman_mh5_support/meshes/mh5l/visual/MH5L_B_AXIS.dae"/>
 				</geometry>
-				<material name="blue"/>
 			</visual>
 			<collision>
-				<!-- <origin rpy="-1.57 0 3.1416" xyz="0 0 0"/> -->
 				<geometry>
-					<mesh filename="package://motoman_mh5_support/meshes/mh5/collision/MH5_B_AXIS.stl" />
+                    <mesh filename="package://motoman_mh5_support/meshes/mh5l/collision/MH5L_B_AXIS.stl" />
 				</geometry>
-				<material name="yellow"/>
 			</collision>
             <xacro:cylinder_inertial radius="0.6" length="0.12" mass="${wrist_2_mass}">
@@ -144,13 +116,11 @@
 			<visual>
 				<geometry>
-					<mesh filename="package://motoman_mh5_support/meshes/mh5/visual/MH5_T_AXIS.stl" />
+                    <mesh filename="package://motoman_mh5_support/meshes/mh5l/visual/MH5L_T_AXIS.dae" />
 				</geometry>
-				<material name="silver"/>
 			</visual>
 			<collision>
 				<geometry>
-					<mesh filename="package://motoman_mh5_support/meshes/mh5/collision/MH5_T_AXIS.stl" />
+                    <mesh filename="package://motoman_mh5_support/meshes/mh5l/collision/MH5L_T_AXIS.stl" />
 				</geometry>
-				<material name="yellow"/>
 			</collision>
             <xacro:cylinder_inertial radius="0.6" length="0.12" mass="${wrist_3_mass}">
@@ -177,5 +147,5 @@
 			<parent link="${prefix}link_l"/>
 			<child link="${prefix}link_u"/>
-			<origin xyz="0 0 0.3100" rpy="0 0 0"/>
+            <origin xyz="0 0 0.4000" rpy="0 0 0"/>
 			<axis xyz="0 -1 0" />
       <!-- Old limits: lower="-2.3736" upper="4.4506" The new limits
@@ -189,5 +159,5 @@
 			<parent link="${prefix}link_u"/>
 			<child link="${prefix}link_r"/>
-			<origin xyz="0.0715 0 0.0399" rpy="0 0 0"/>
+            <origin xyz="0.0715 0 0.0400" rpy="0 0 0"/>
 			<axis xyz="-1 0 0" />
 			<limit lower="-3.3161" upper="3.3161" effort="100" velocity="3.48" />
@@ -196,5 +166,5 @@
 			<parent link="${prefix}link_r"/>
 			<child link="${prefix}link_b"/>
-			<origin xyz="0.2335 0 0" rpy="0 0 0"/>
+            <origin xyz="0.3335 0 0" rpy="0 0 0"/>
 			<axis xyz="0 -1 0" />
 			<limit lower="-2.1817" upper="2.1817" effort="100" velocity="3.48" />
@@ -203,5 +173,5 @@
 			<parent link="${prefix}link_b"/>
 			<child link="${prefix}link_t"/>
-			<origin xyz="0.0865 0 0" rpy="0 0 0"/>
+            <origin xyz="0.0800 0 0" rpy="0 0 0"/>
 			<axis xyz="-1 0 0" />
 			<limit lower="-6.2831" upper="6.2831" effort="100" velocity="6.97" />

Commit message: used jog to modify urdf joint limits, Marq's threading fix and added errors

File: motoman_mh5_support/urdf/mh5l_macro.xacro (robot description, xacro)
@@ -135,5 +135,5 @@
 			<origin xyz="0 0 0.1990" rpy="0 0 0"/>
 			<axis xyz="0 0 1" />
-			<limit lower="-2.9671" upper="2.9671" effort="100" velocity="2.96" />
+      <limit lower="-2.96" upper="2.96" effort="100" velocity="2.96" />
 		</joint>
 		<joint name="${prefix}joint_l" type="revolute">
@@ -142,5 +142,5 @@
 			<origin xyz="0.0880 0 0.1310" rpy="0 0 0"/>
 			<axis xyz="0 1 0" />
-			<limit lower="-1.1345" upper="2.6180" effort="100" velocity="2.96" />
+      <limit lower="-1.13" upper="2.26" effort="100" velocity="2.96" />
 		</joint>
 		<joint name="${prefix}joint_u" type="revolute">
@@ -154,5 +154,6 @@
            old limits were converted directly from the MH5 data sheet,
            which was clearly way off. -->
-			<limit lower="-1.0122" upper="3.2218" effort="100" velocity="2.96" />
+      <!--<limit lower="-1.0122" upper="3.2218" effort="100" velocity="2.96" />-->
+      <limit lower="-1.0122" upper="2.0" effort="100" velocity="2.96" />
 		</joint>
 		<joint name="${prefix}joint_r" type="revolute">
@@ -161,5 +162,5 @@
             <origin xyz="0.0715 0 0.0400" rpy="0 0 0"/>
 			<axis xyz="-1 0 0" />
-			<limit lower="-3.3161" upper="3.3161" effort="100" velocity="3.48" />
+      <limit lower="-3.31" upper="3.31" effort="100" velocity="3.48" />
 		</joint>
 		<joint name="${prefix}joint_b" type="revolute">
@@ -168,5 +169,5 @@
             <origin xyz="0.3335 0 0" rpy="0 0 0"/>
 			<axis xyz="0 -1 0" />
-			<limit lower="-2.1817" upper="2.1817" effort="100" velocity="3.48" />
+      <limit lower="-2.06" upper="2.1" effort="100" velocity="3.48" />
 		</joint>
 		<joint name="${prefix}joint_t" type="revolute">
@@ -175,5 +176,6 @@
             <origin xyz="0.0800 0 0" rpy="0 0 0"/>
 			<axis xyz="-1 0 0" />
-			<limit lower="-6.2831" upper="6.2831" effort="100" velocity="6.97" />
+      <!--<limit lower="-6.2831" upper="6.2831" effort="100" velocity="6.97" />-->
+      <limit lower="-4.0" upper="4.0" effort="100" velocity="6.97" />
 		</joint>
 		<!-- end of joint list -->
