Commit message: Final moveit config

File: motoman_es165d_support/urdf/es165d_macro.xacro (robot description, xacro)
@@ -63,4 +63,40 @@
         </collision>
     </link>
+    <link name="${prefix}B_axis">
+        <visual>
+            <geometry>
+                <mesh filename="package://motoman_es165d_support/meshes/visual/B_axis.dae"/>
+            </geometry>
+        </visual>
+        <collision>
+            <geometry>
+                <mesh filename="package://motoman_es165d_support/meshes/collision/B_axis.stl"/>
+            </geometry>
+        </collision>
+    </link>
+    <link name="${prefix}T_axis">
+        <visual>
+            <geometry>
+                <mesh filename="package://motoman_es165d_support/meshes/visual/T_axis.dae"/>
+            </geometry>
+        </visual>
+        <collision>
+            <geometry>
+                <mesh filename="package://motoman_es165d_support/meshes/collision/T_axis.stl"/>
+            </geometry>
+        </collision>
+    </link>
+    <link name="${prefix}CWeight">
+        <visual>
+            <geometry>
+                <mesh filename="package://motoman_es165d_support/meshes/visual/CWeight.dae"/>
+            </geometry>
+        </visual>
+        <collision>
+            <geometry>
+                <mesh filename="package://motoman_es165d_support/meshes/collision/CWeight.stl"/>
+            </geometry>
+        </collision>
+    </link>
     <!-- end of link list -->
     <!-- joint list -->
@@ -70,5 +106,5 @@
         <origin xyz="0 0 0.302" rpy="0 0 0" />
         <axis xyz="0 0 1" />
-        <limit lower="-2.9670" upper="2.9670" effort="212.66" velocity="6.5448"/>
+        <limit lower="${-pi}" upper="${pi}" effort="212.66" velocity="1.92"/>
     </joint>
     <joint name="${prefix}joint_2_l" type="revolute">
@@ -77,5 +113,5 @@
         <origin xyz="0.285 -0.082 0.348" rpy="${pi/2} 0 ${pi}" />
         <axis xyz="0 0 1" />
-        <limit lower="-2.9670" upper="2.9670" effort="212.66" velocity="6.5448"/>
+        <limit lower="-1.07" upper="1.35" effort="212.66" velocity="1.92"/>
     </joint>
     <joint name="${prefix}joint_3_u" type="revolute">
@@ -84,12 +120,31 @@
         <origin xyz="0 1.150 -0.235" rpy="0 0 0" />
         <axis xyz="0 0 1" />
-        <limit lower="-2.9670" upper="2.9670" effort="212.66" velocity="6.5448"/>
+        <limit lower="-1.89" upper="2.97" effort="212.66" velocity="1.92"/>
     </joint>
     <joint name="${prefix}joint_4_r" type="revolute">
         <parent link="${prefix}U_axis"/>
         <child link="${prefix}R_axis"/>
-        <origin xyz="1.225 -0.25 317" rpy="0 0 0" />
+        <origin xyz="0.25 1.225 0.317" rpy="${-pi/2} 0 0" />
         <axis xyz="0 0 1" />
-        <limit lower="-2.9670" upper="2.9670" effort="212.66" velocity="6.5448"/>
+        <limit lower="-3.57792" upper="3.57792" effort="212.66" velocity="3.05"/>
+    </joint>
+    <joint name="${prefix}joint_5_b" type="revolute">
+        <parent link="${prefix}R_axis"/>
+        <child link="${prefix}B_axis"/>
+        <origin xyz="0 0 0" rpy="0 ${-pi/2} ${pi/2}" />
+        <axis xyz="0 0 1" />
+        <limit lower="-2.0944" upper="2.0944" effort="212.66" velocity="2.53"/>
+    </joint>
+    <joint name="${prefix}joint_6_t" type="revolute">
+        <parent link="${prefix}B_axis"/>
+        <child link="${prefix}T_axis"/>
+        <origin xyz="0 0 0" rpy="0 ${pi/2} 0" />
+        <axis xyz="0 0 1" />
+        <limit lower="-3.49" upper="3.49" effort="212.66" velocity="4.19"/>
+    </joint>
+    <joint name="${prefix}joint_2_cw" type="fixed">
+        <parent link="${prefix}S_axis"/>
+        <child link="${prefix}CWeight"/>
+        <origin xyz="-0.32 0.0362 0.3381" rpy=" ${pi/2} 0 0" />
     </joint>
     <!-- ROS base_link to Robot Manufacturer World Coordinates transform -->
@@ -102,2 +157,3 @@
     </xacro:macro>
 </robot>
+<!--/home/stephen/motoman_ws/src/motoman/motoman_es165d_support/urdf/es165d.xacro-->

Commit message: updated URDF based on DH parameters from ALL.PRM file

File: motoman_es165d_support/urdf/es165d_macro.xacro (robot description, xacro)
@@ -134,5 +134,5 @@
       <origin xyz="0 0 0.650" rpy="0 0 0"/>
       <axis xyz="0 0 1" />
-      <limit lower="-${pi}" upper="${pi}" effort="100" velocity="1.83" />
+      <limit lower="-${pi}" upper="${pi}" effort="10000" velocity="1.92" />
 		</joint>
 		<joint name="${prefix}joint_l" type="revolute">
@@ -140,6 +140,6 @@
 			<child link="${prefix}link_l"/>
       <origin xyz="0.285 0 0" rpy="0 0 0"/>
-      <axis xyz="0 -1 0" />
-      <limit lower="-2.268" upper="1.396" effort="100" velocity="1.83" />
+      <axis xyz="0 1 0" />
+      <limit lower="-1.04" upper="1.32" effort="10000" velocity="1.92" />
 		</joint>
 		<joint name="${prefix}joint_u" type="revolute">
@@ -148,5 +148,5 @@
       <origin xyz="0 0 1.150" rpy="0 0 0"/>
       <axis xyz="0 -1 0" />
-      <limit lower="-1.46" upper="4.12" effort="100" velocity="1.83" />
+      <limit lower="-1.41" upper="3.43" effort="10000" velocity="1.92" />
 		</joint>
 		<joint name="${prefix}joint_r" type="revolute">
@@ -155,5 +155,5 @@
       <origin xyz="1.225 0 0.250" rpy="0 0 0"/>
 			<axis xyz="-1 0 0" />
-      <limit lower="-${2*pi}" upper="${2*pi}" effort="100" velocity="3.05" />
+      <limit lower="-6.2" upper="6.2" effort="10000" velocity="3.05" />
 		</joint>
 		<joint name="${prefix}joint_b" type="revolute">
@@ -162,5 +162,5 @@
       <origin xyz="0 0 0" rpy="0 0 0"/>
 			<axis xyz="0 -1 0" />
-      <limit lower="-2.268" upper="2.268" effort="100" velocity="2.61" />
+      <limit lower="-2.26" upper="2.26" effort="10000" velocity="2.62" />
 		</joint>
 		<joint name="${prefix}joint_t" type="revolute">
@@ -169,5 +169,5 @@
             <origin xyz="0.225 0 0" rpy="0 0 0"/>
 			<axis xyz="-1 0 0" />
-      <limit lower="-${2*pi}" upper="${2*pi}" effort="100" velocity="4.18" />
+      <limit lower="-${2*pi}" upper="${2*pi}" effort="10000" velocity="4.18" />
 		</joint>
 		<!-- end of joint list -->

Commit message: reduced joint r and t motion to +-180

File: motoman_es165d_support/urdf/es165d_macro.xacro (robot description, xacro)
@@ -155,5 +155,5 @@
       <origin xyz="1.225 0 0.250" rpy="0 0 0"/>
 			<axis xyz="-1 0 0" />
-      <limit lower="-6.2" upper="6.2" effort="10000" velocity="3.05" />
+      <limit lower="-${pi}" upper="${pi}" effort="10000" velocity="3.05" />
 		</joint>
 		<joint name="${prefix}joint_b" type="revolute">
@@ -169,5 +169,5 @@
             <origin xyz="0.225 0 0" rpy="0 0 0"/>
 			<axis xyz="-1 0 0" />
-      <limit lower="-${2*pi}" upper="${2*pi}" effort="10000" velocity="4.18" />
+      <limit lower="-${pi}" upper="${pi}" effort="10000" velocity="4.18" />
 		</joint>
 		<!-- end of joint list -->
