Commit message: added es165d-100 fast IK and es165d URDF documentation

File: motoman_es165d_support/urdf/es165d_100_macro.xacro (robot description, xacro)
@@ -169,5 +169,5 @@
             <origin xyz="0.225 0 0" rpy="0 0 0"/>
 			<axis xyz="-1 0 0" />
-      <limit lower="-${pi}" upper="${pi}" effort="10000" velocity="4.18" />
+      <limit lower="-${pi}" upper="${pi}" effort="10000" velocity="4.19" />
 		</joint>
 		<!-- end of joint list -->
